File: rev1/6502-rev1.kicad_pcb (KiCad board)
At the start: 2 copper layers, 172 x 136 mm, 57 parts, among them J1 DC Jack, J2 CLK_HDR, J3 LCD Socket, J4 DB9_Female, J5 65C02 Debug Port, SW1 PWR_SWITCH, SW3 ENTER, SW4 UP, SW5 DOWN, SW6 LEFT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

Commit message: Update rev1.0
Parts:
- added R13: 3.3k, Resistor_THT:R_Axial_DIN0207_L6.3mm_D2.5mm_P7.62mm_Horizontal, F.Cu at (97.0, 95.5)
- C2: value 0.1uF -> 0.1 uF
- moved SW2 24.0 mm to (101.8, 128.8)
- moved RV1 9.50 mm to (105.0, 152.0)
- renumbered CONTRAST to RV1, RESET to SW2
Connections:
- C3 pad 1: Net-(C3-Pad1) -> GND
- R1 pad 2: Net-(C3-Pad1) -> ~{RES}
- SW2 pad 1: Net-(C3-Pad1) -> GND
- U2 pad 38: unconnected-(U2-~{SO}-Pad38) -> Net-(U2-~{SO})
Routing:
- net Net-(C3-Pad1): track 242.7 -> 0.00 mm
- net CLK: track 241.1 -> 294.5 mm, vias 4 -> 1
- net +5V: track 577.1 -> 625.9 mm, vias 0 -> 1
- net Net-(U2-~{SO}): track 0.00 -> 44.4 mm
- net CLK_OUT: track 176.6 -> 217.9 mm, vias 0 -> 1
- net ~{RES}: track 266.2 -> 298.4 mm, vias 1 -> 3
- net ~{R/W}: track 197.2 -> 229.4 mm, vias 2 -> 1
- net a14: track 260.8 -> 229.7 mm, vias 1 -> 2
- net a10: track 206.8 -> 175.8 mm, vias 3 -> 1
- net d3: track 228.4 -> 200.3 mm, vias 0 -> 3
- net GND: track 604.5 -> 630.0 mm
- net a15: track 158.4 -> 183.3 mm, vias 2 -> 1
- net CS_IO: track 129.1 -> 153.6 mm
- net a13: track 208.6 -> 187.7 mm, vias 1 -> 4
- net d4: track 198.1 -> 217.9 mm, vias 0 -> 2
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- added copper zone on B.Cu, net GND
- added copper zone on F.Cu, net GND
Other:
- board text added: "CONTRAST"
