File: rev1/6502-rev1.kicad_sch (KiCad schematic)
At the start: 54 parts, among them J1 DC Jack, J2 CLK_HDR, J3 LCD Socket, J4 DB9_Female, J5 65C02 Debug Port, SW1 PWR_SWITCH, SW2 RESET, SW3 ENTER, SW4 UP, SW5 DOWN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

Commit message: Update rev1.0
Parts:
- added R13: 3.3k, Resistor_THT:R_Axial_DIN0207_L6.3mm_D2.5mm_P7.62mm_Horizontal, symbol Device:R
- C4: footprint SamacSys_Parts:C322C104K1R5TA -> SamacSys_Parts:C322C104K1R5TA
Connections:
- net +5V: now also R13.1
- net GND: now also C3.1, SW2.1
- net ~{RES}: now also R1.2
- net at U2.38 (~{SO}): now also R13.2
- no-connect marks 34 -> 33
Other:
- moved on the sheet: C3, R1, SW2
